File: Controller.kicad_sch (KiCad schematic)
At the start: 46 parts, among them J1 USB4105-GF-A-060, J2 BM03B-SRSS-TB, J3 SWD 2.54 DNP, SW61 BOOTSEL, SW62 RESET, U1 RP2354A, U2 XC6206P332MR-G, U3 USBLC6-2SC6, X1 12MHz

Commit message: Add side LEDs and preserve verified official core routing
Other:
- note added: "TP2：GPIO17の3.3 Vデータ。R24（100Ω）経由でサイドLEDを駆動。"
- note removed: "TP2は3.3 V GPIO。5 V LEDドライバは搭載しない。"
Changed lines of the file:
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@@
 		(property
 "Description"
-"Expansion pads only. LED not fitted; GPIO is 3.3V, not a 5V NeoPixel driver."
+"VBUS power test pad; shared 5V USB rail for the side LEDs"
 			(at 54.61 193.04 0)
 			(effects
@@
 		(property
 "Description"
-"Expansion pads only. LED not fitted; GPIO is 3.3V, not a 5V NeoPixel driver."
+"GPIO17 3.3V LED data test point; R24 100ohm drives the first WS2812B-4020-V6 DIN directly."
 			(at 294.64 248.92 0)
 			(effects
@@
 		(property
 "Description"
-"Expansion pads only. LED not fitted; GPIO is 3.3V, not a 5V NeoPixel driver."
+"GND reference test pad"
 			(at 82.55 193.04 0)
 			(effects
@@
 					(reference "X1")
 					(unit 1)))))
-	(label
+	(global_label
 "GND"
+		(shape bidirectional)
 		(at 255.27 179.07 0)
 		(effects
@@
 			(justify left bottom))
 )
-	(label
+	(global_label
 "GND"
+		(shape bidirectional)
 		(at 355.6 128.27 0)
 		(effects
@@
 			(justify left bottom))
 )
-	(label
+	(global_label
 "GND"
+		(shape bidirectional)
 		(at 328.93 110.49 0)
 		(effects
@@
 			(justify right bottom))
 )
-	(label
+	(global_label
 "GND"
+		(shape bidirectional)
 		(at 231.14 46.99 0)
 		(effects
@@
 			(justify left bottom))
 )
-	(label
+	(global_label
 "GND"
+		(shape bidirectional)
 		(at 367.03 45.72 0)
 		(effects
@@
 			(justify left bottom))
 )
-	(label
+	(global_label
 "GND"
+		(shape bidirectional)
 		(at 228.6 247.65 0)
 		(effects
@@
 			(justify left bottom))
 )
-	(label
+	(global_label
 "GND"
+		(shape bidirectional)
 		(at 170.18 184.15 0)
 		(effects
@@
 			(justify left bottom))
 )
-	(label
+	(global_label
 "GND"
+		(shape bidirectional)
 		(at 365.76 219.71 0)
 		(effects
@@
 			(justify left bottom))
 )
-	(label
+	(global_label
 "GND"
+		(shape bidirectional)
 		(at 321.31 248.92 0)
 		(effects
@@
 			(justify left bottom))
 )
-	(label
+	(global_label
 "VBUS"
+		(shape bidirectional)
 		(at 109.22 68.58 180)
 		(effects
@@
 			(justify right bottom))
 )
-	(label
+	(global_label
 "GND"
+		(shape bidirectional)
 		(at 109.22 101.6 180)
 		(effects
@@
 			(justify right bottom))
 )
-	(label
+	(global_label
 "VBUS"
+		(shape bidirectional)
 		(at 55.88 76.2 180)
 		(effects
@@
 			(justify right bottom))
 )
-	(label
+	(global_label
 "GND"
+		(shape bidirectional)
 		(at 68.58 121.92 180)
 		(effects
@@
 			(justify right bottom))
 )
-	(label
+	(global_label
 "VBUS"
+		(shape bidirectional)
 		(at 54.61 43.18 0)
 		(effects
@@
 			(justify left bottom))
 )
-	(label
+	(global_label
 "GND"
+		(shape bidirectional)
 		(at 77.47 59.69 0)
 		(effects
@@
 			(justify left bottom))
 )
-	(label
+	(global_label
 "VBUS"
+		(shape bidirectional)
 		(at 54.61 189.23 0)
 		(effects
@@
 			(justify left bottom))
 )
-	(label
+	(global_label
 "GND"
+		(shape bidirectional)
 		(at 82.55 196.85 0)
 		(effects
@@
 			(justify left bottom))
 )
-	(label
+	(global_label
 "VBUS"
+		(shape bidirectional)
 		(at 40.64 40.64 0)
 		(effects
@@
 			(justify left bottom))
 )
-	(label
+	(global_label
 "GND"
+		(shape bidirectional)
 		(at 40.64 59.69 0)
 		(effects
@@
 			(justify left bottom))
 )
-	(label
+	(global_label
 "GND"
+		(shape bidirectional)
 		(at 358.14 238.76 0)
 		(effects
@@
 			(justify left bottom))
 )
-	(label
+	(global_label
 "EXP_GPIO17_3V3"
+		(shape bidirectional)
 		(at 294.64 248.92 0)
 		(effects
@@
 )
 	(text
-"TP2は3.3 V GPIO。5 V LEDドライバは搭載しない。"
+"TP2：GPIO17の3.3 Vデータ。R24（100Ω）経由でサイドLEDを駆動。"
 		(at 15.24 278.13 0)
 		(effects

Commit message: Apply delivered LCSC procurement assignments
Parts:
- C10, C6, C7, C9: LCSC (none) -> C82453; manufacturer Murata -> Murata Electronics
- C11, C12, C13, C14, C15, C16, C17, C18, C20, C21, C8: LCSC (none) -> C307331; manufacturer Murata -> Samsung Electro-Mechanics; manufacturer_pn GRM155R71E104KE14D -> CL05B104KB54PNC; voltage 25V -> 50V
- C3, C4: LCSC (none) -> C1548; manufacturer Murata -> FH (Guangdong Fenghua Advanced Tech); manufacturer_pn GRM1555C1H150JA01D -> 0402CG150J500NT
- J2: LCSC C5306067 -> C160389
- L1: LCSC (none) -> C42411119
- R2, R4, R6: LCSC (none) -> C11702; manufacturer Yageo -> UNI-ROYAL(Uniroyal Elec); manufacturer_pn RC0402FR-071KL -> 0402WGF1001TCE
- R20, R21: LCSC (none) -> C25905; manufacturer Yageo -> UNI-ROYAL(Uniroyal Elec); manufacturer_pn RC0402FR-075K1L -> 0402WGF5101TCE
- R22, R23: LCSC (none) -> C25076; manufacturer Yageo -> UNI-ROYAL(Uniroyal Elec); manufacturer_pn RC0402FR-07100RL -> 0402WGF1000TCE
- R3: LCSC (none) -> C25105; manufacturer Yageo -> UNI-ROYAL(Uniroyal Elec); manufacturer_pn RC0402FR-0733RL -> 0402WGF330JTCE
- R7, R8: LCSC (none) -> C25100; manufacturer Yageo -> UNI-ROYAL(Uniroyal Elec); manufacturer_pn RC0402FR-0727RL -> 0402WGF270JTCE
- U1: LCSC (none) -> C41378174
- X1: LCSC (none) -> C20625731
