File: LEDs.kicad_sch (KiCad schematic)
At the start: 49 parts

Commit message: Apply delivered LCSC procurement assignments
Parts:
- C22, C23, C24, C25, C26, C27, C28, C29, C30, C31, C32, C33, C34, C35, C36, C37: LCSC (none) -> C307331; manufacturer Murata -> Samsung Electro-Mechanics; manufacturer_pn GRM155R71E104KE14D -> CL05B104KB54PNC; voltage 25V -> 50V
- R24: LCSC (none) -> C25076; manufacturer Yageo -> UNI-ROYAL(Uniroyal Elec); manufacturer_pn RC0402FR-07100RL -> 0402WGF1000TCE
