File: WING27.kicad_sch (KiCad schematic)
At the start: 60 parts, among them SW1 Kailh_CMI627301D60, SW10 Kailh_CMI627301D60, SW11 Kailh_CMI627301D60, SW12 Kailh_CMI627301D60, SW13 Kailh_CMI627301D60, SW14 Kailh_CMI627301D60, SW15 Kailh_CMI627301D60, SW16 Kailh_CMI627301D60, SW17 Kailh_CMI627301D60, SW18 Kailh_CMI627301D60, SW19 Kailh_CMI627301D60, SW2 Kailh_CMI627301D60, SW20 Kailh_CMI627301D60, SW21 Kailh_CMI627301D60, SW22 Kailh_CMI627301D60, SW23 Kailh_CMI627301D60, SW24 Kailh_CMI627301D60, SW25 Kailh_CMI627301D60, SW26 Kailh_CMI627301D60, SW27 Kailh_CMI627301D60, SW28 Kailh_CMI627301D60, SW29 Kailh_CMI627301D60, SW3 Kailh_CMI627301D60, SW30 Kailh_CMI627301D60, SW31 Kailh_CMI627301D60, SW32 Kailh_CMI627301D60, SW33 Kailh_CMI627301D60, SW34 Kailh_CMI627301D60, SW35 Kailh_CMI627301D60, SW36 Kailh_CMI627301D60, SW37 Kailh_CMI627301D60, SW38 Kailh_CMI627301D60, SW39 Kailh_CMI627301D60, SW4 Kailh_CMI627301D60, SW40 Kailh_CMI627301D60, SW41 Kailh_CMI627301D60, SW42 Kailh_CMI627301D60, SW43 Kailh_CMI627301D60, SW44 Kailh_CMI627301D60, SW45 Kailh_CMI627301D60, SW46 Kailh_CMI627301D60, SW47 Kailh_CMI627301D60, SW48 Kailh_CMI627301D60, SW49 Kailh_CMI627301D60, SW5 Kailh_CMI627301D60, SW50 Kailh_CMI627301D60, SW51 Kailh_CMI627301D60, SW52 Kailh_CMI627301D60, SW53 Kailh_CMI627301D60, SW54 Kailh_CMI627301D60, SW55 Kailh_CMI627301D60, SW56 Kailh_CMI627301D60, SW57 Kailh_CMI627301D60, SW58 Kailh_CMI627301D60, SW59 Kailh_CMI627301D60, SW6 Kailh_CMI627301D60, SW60 Kailh_CMI627301D60, SW7 Kailh_CMI627301D60, SW8 Kailh_CMI627301D60, SW9 Kailh_CMI627301D60

Commit message: Complete WING27 electrical design and verified footprints before routing
Parts:
- added D1, D10, D11, D12, D13, D14, D15, D16, D17, D18, D19, D2, D20, D21, D22, D23, D24, D25, D26, D27, D28, D29, D3, D30, D4, D5, D6, D7, D8, D9: BAV70, WING27:SOT-23, symbol WING27:BAV70
- SW1, SW10, SW11, SW12, SW14, SW15, SW16, SW17, SW18, SW19, SW2, SW20, SW21, SW22, SW23, SW24, SW25, SW26, SW27, SW28, SW3, SW30, SW31, SW32, SW33, SW34, SW35, SW36, SW37, SW38, SW39, SW4, SW40, SW41, SW42, SW43, SW44, SW45, SW46, SW47, SW48, SW49, SW5, SW50, SW51, SW52, SW53, SW54, SW55, SW56, SW57, SW58, SW59, SW6, SW60, SW7, SW8, SW9: value Kailh_CMI627301D60 -> CMI627301D60; MPN CMI627301D60 -> (none); Manufacturer Kailh -> (none); Operating Force 60+/-15 gf -> (none); manufacturer (none) -> Kailh; manufacturer_pn (none) -> CMI627301D60
- SW13, SW29: value Kailh_CMI627301D60 -> CMI627301D60; Legend (blank) -> (none); MPN CMI627301D60 -> (none); Manufacturer Kailh -> (none); Operating Force 60+/-15 gf -> (none); manufacturer (none) -> Kailh; manufacturer_pn (none) -> CMI627301D60
Connections:
- net COL3: now reaches SW4.1
- net COL3: now also SW10.1, SW16.1, SW22.1, SW28.1
- net KEY_L1_4: now reaches SW4.2
- net KEY_L1_4: now also D2.2 (A)
- net COL9: now reaches SW58.1
- net COL9: now also SW34.1, SW41.1, SW47.1, SW52.1
- net KEY_R5_4: now reaches SW58.2
- net KEY_R5_4: now also D29.2 (A)
- net COL8: now reaches SW57.1
- net COL8: now also SW33.1, SW40.1, SW46.1, SW51.1
- net KEY_R5_3: now reaches SW57.2
- net KEY_R5_3: now also D29.1 (A)
- net COL0: now reaches SW19.1
- net COL0: now also SW1.1, SW13.1, SW25.1, SW7.1
- net KEY_L4_1: now reaches SW19.2
- net KEY_L4_1: now also D19.1 (A)
- net KEY_R4_3: now reaches SW51.2
- net KEY_R4_3: now also D23.1 (A)
- net COL6: now reaches SW55.1
- net COL6: now also SW31.1, SW38.1, SW44.1, SW49.1
- net KEY_R5_1: now reaches SW55.2
- net KEY_R5_1: now also D28.1 (A)
- net COL11: now reaches SW48.1
- net COL11: now also SW36.1, SW43.1, SW54.1, SW60.1
- net KEY_R3_5: now reaches SW48.2
- net KEY_R3_5: now also D18.2 (A)
- net COL2: now reaches SW3.1
- net COL2: now also SW15.1, SW21.1, SW27.1, SW9.1
- net KEY_L1_3: now reaches SW3.2
- net KEY_L1_3: now also D2.1 (A)
- net COL1: now reaches SW8.1
- net COL1: now also SW14.1, SW2.1, SW20.1, SW26.1
- net KEY_L2_2: now reaches SW8.2
- net KEY_L2_2: now also D7.2 (A)
- net COL4: now reaches SW23.1
- net COL4: now also SW11.1, SW17.1, SW29.1, SW5.1
- net KEY_L4_5: now reaches SW23.2
- net KEY_L4_5: now also D21.1 (A)
- net KEY_L1_1: now reaches SW1.2
- net KEY_L1_1: now also D1.1 (A)
- net KEY_L3_4: now reaches SW16.2
- net KEY_L3_4: now also D14.2 (A)
- net KEY_R5_6: now reaches SW60.2
- net KEY_R5_6: now also D30.2 (A)
- net COL7: now reaches SW56.1
- net COL7: now also SW32.1, SW39.1, SW45.1, SW50.1
- net KEY_R5_2: now reaches SW56.2
- net KEY_R5_2: now also D28.2 (A)
- net KEY_R1_2: now reaches SW32.2
- net KEY_R1_2: now also D4.2 (A)
- net KEY_L5_2: now reaches SW26.2
- net KEY_L5_2: now also D25.2 (A)
- net KEY_R1_4: now reaches SW34.2
- net KEY_R1_4: now also D5.2 (A)
- net COL5: now reaches SW12.1
- net COL5: now also SW18.1, SW24.1, SW30.1, SW6.1
- net KEY_L2_6: now reaches SW12.2
- net KEY_L2_6: now also D9.2 (A)
- net KEY_L1_2: now reaches SW2.2
- net KEY_L1_2: now also D1.2 (A)
- net KEY_L3_6: now reaches SW18.2
- net KEY_L3_6: now also D15.2 (A)
- net KEY_L5_4: now reaches SW28.2
- net KEY_L5_4: now also D26.2 (A)
- net KEY_R1_3: now reaches SW33.2
- net KEY_R1_3: now also D5.1 (A)
- net KEY_L1_6: now reaches SW6.2
- net KEY_L1_6: now also D3.2 (A)
- net KEY_L3_3: now reaches SW15.2
- net KEY_L3_3: now also D14.1 (A)
- net KEY_L4_6: now reaches SW24.2
- net KEY_L4_6: now also D21.2 (A)
- net KEY_L2_3: now reaches SW9.2
- net KEY_L2_3: now also D8.1 (A)
- net KEY_R4_4: now reaches SW52.2
- net KEY_R4_4: now also D23.2 (A)
- net COL10: now reaches SW42.1
- net COL10: now also SW35.1, SW37.1, SW53.1, SW59.1
- net KEY_R2_5: now reaches SW42.2
- net KEY_R2_5: now also D18.1 (A)
- net KEY_R4_2: now reaches SW50.2
- net KEY_R4_2: now also D22.2 (A)
- net KEY_L5_5: now reaches SW29.2
- net KEY_L5_5: now also D27.1 (A)
- net KEY_R1_5: now reaches SW35.2
- net KEY_R1_5: now also D6.1 (A)
- net KEY_L1_5: now reaches SW5.2
- net KEY_L1_5: now also D3.1 (A)
- net KEY_R5_5: now reaches SW59.2
- net KEY_R5_5: now also D30.1 (A)
- net KEY_R4_6: now reaches SW54.2
- net KEY_R4_6: now also D24.2 (A)
- net KEY_R3_2: now reaches SW45.2
- net KEY_R3_2: now also D16.2 (A)
- net KEY_L3_5: now reaches SW17.2
- net KEY_L3_5: now also D15.1 (A)
- net KEY_L5_6: now reaches SW30.2
- net KEY_L5_6: now also D27.2 (A)
- net KEY_R2_2: now reaches SW39.2
- net KEY_R2_2: now also D10.2 (A)
- net KEY_R4_5: now reaches SW53.2
- net KEY_R4_5: now also D24.1 (A)
- net KEY_R4_1: now reaches SW49.2
- net KEY_R4_1: now also D22.1 (A)
- net KEY_L5_3: now reaches SW27.2
- net KEY_L5_3: now also D26.1 (A)
- net KEY_L2_1: now reaches SW7.2
- net KEY_L2_1: now also D7.1 (A)
- net KEY_R2_4: now reaches SW41.2
- net KEY_R2_4: now also D11.2 (A)
- net KEY_R2_6: now reaches SW43.2
- net KEY_R2_6: now also D12.2 (A)
- net KEY_L5_1: now reaches SW25.2
- net KEY_L5_1: now also D25.1 (A)
- net KEY_L4_4: now reaches SW22.2
- net KEY_L4_4: now also D20.2 (A)
- net KEY_L3_2: now reaches SW14.2
- net KEY_L3_2: now also D13.2 (A)
- net KEY_R1_1: now reaches SW31.2
- net KEY_R1_1: now also D4.1 (A)
- net KEY_L2_4: now reaches SW10.2
- net KEY_L2_4: now also D8.2 (A)
- net KEY_R2_3: now reaches SW40.2
- net KEY_R2_3: now also D11.1 (A)
- net KEY_R3_1: now reaches SW44.2
- net KEY_R3_1: now also D16.1 (A)
- net KEY_R2_1: now reaches SW38.2
- net KEY_R2_1: now also D10.1 (A)
- net KEY_L4_2: now reaches SW20.2
- net KEY_L4_2: now also D19.2 (A)
- net KEY_R1_7: now reaches SW37.2
- net KEY_R1_7: now also D12.1 (A)
- net KEY_R3_4: now reaches SW47.2
- net KEY_R3_4: now also D17.2 (A)
- net KEY_L3_1: now reaches SW13.2
- net KEY_L3_1: now also D13.1 (A)
- net KEY_L2_5: now reaches SW11.2
- net KEY_L2_5: now also D9.1 (A)
- net KEY_R1_6: now reaches SW36.2
- net KEY_R1_6: now also D6.2 (A)
- net KEY_L4_3: now reaches SW21.2
- net KEY_L4_3: now also D20.1 (A)
- net KEY_R3_3: now reaches SW46.2
- net KEY_R3_3: now also D17.1 (A)
- new net ROW0: D1.3 (K), D2.3 (K), D3.3 (K), D4.3 (K), D5.3 (K), D6.3 (K)
- new net ROW1: D10.3 (K), D11.3 (K), D12.3 (K), D7.3 (K), D8.3 (K), D9.3 (K)
- new net ROW2: D13.3 (K), D14.3 (K), D15.3 (K), D16.3 (K), D17.3 (K), D18.3 (K)
- new net ROW3: D19.3 (K), D20.3 (K), D21.3 (K), D22.3 (K), D23.3 (K), D24.3 (K)
- new net ROW4: D25.3 (K), D26.3 (K), D27.3 (K), D28.3 (K), D29.3 (K), D30.3 (K)
Other:
- added sheet Controller (Controller.kicad_sch)
- note added: "60 keys / 5 rows x 12 columns. Read COL0..11 with pull-ups; drive one ROW low, other ROWs high-impedance."
- note added: "BAV70: pin 1/2 = independent anodes; pin 3 = common cathode to one ROW. Physical stagger is independent of logical row."
- note added: "L3_1 /"
- note added: "L5_5 /"
- note removed: "All 60 switches, including L3_1 and L5_5, are retained. Open pins are intentional pending circuit definition."
- note removed: "L3_1 / (blank)"
- note removed: "L5_5 / (blank)"
- note removed: "P2 coordinates and switch geometry verified. Controller / matrix / USB-C / PCB outline pending confirmation."
- title: WING27 P2 / 60-key verified placement -> WING27 / 60-key matrix
- moved on the sheet: SW1, SW10, SW11, SW12, SW13, SW14, SW15, SW16, SW17, SW18, SW19, SW2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

Commit message: Refine WING27 schematics, SWD connector, panel overlay and mounting
Other:
- note added: "60-key matrix / COL0..11 input with pull-ups; selected ROW low, other ROWs high-impedance"
- note added: "BAV70: independent anodes 1 / 2; common cathode 3. Dots are connections; unmarked bus crossings are not connected."
- note added: "L3_1 / (blank)"
- note added: "L5_5 / (blank)"
- note added: "Logical rows preserve all 60 physical key IDs; staggered right-hand rows use nearby two-key pairs."
- note removed: "60 keys / 5 rows x 12 columns. Read COL0..11 with pull-ups; drive one ROW low, other ROWs high-impedance."
- note removed: "BAV70: pin 1/2 = independent anodes; pin 3 = common cathode to one ROW. Physical stagger is independent of logical row."
- note removed: "L3_1 /"
- note removed: "L5_5 /"
- company: (none) -> ハシビロ工業
- moved on the sheet: D1, D10, D11, D12, D13, D14, D15, D16, D17, D18, D19, D2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

Commit message: Split keyboard GPIO banks and refine basic parts and SWD options
Connections:
- net ROW0 renamed ROW_L0
- net ROW_L0: no longer D4.3 (K), D5.3 (K), D6.3 (K)
- net ROW1 renamed ROW_L1
- net ROW_L1: no longer D10.3 (K), D11.3 (K), D12.3 (K)
- net ROW2 renamed ROW_L2
- net ROW_L2: no longer D16.3 (K), D17.3 (K), D18.3 (K)
- net ROW3 renamed ROW_L3
- net ROW_L3: no longer D22.3 (K), D23.3 (K), D24.3 (K)
- net ROW4 renamed ROW_L4
- net ROW_L4: no longer D28.3 (K), D29.3 (K), D30.3 (K)
- new net ROW_R0: D4.3 (K), D5.3 (K), D6.3 (K)
- new net ROW_R1: D10.3 (K), D11.3 (K), D12.3 (K)
- new net ROW_R2: D16.3 (K), D17.3 (K), D18.3 (K)
- new net ROW_R3: D22.3 (K), D23.3 (K), D24.3 (K)
- new net ROW_R4: D28.3 (K), D29.3 (K), D30.3 (K)
Other:
- note added: "Two independent 5x6 matrices / COL0..5 left, COL6..11 right / separate ROW_L and ROW_R"
- note removed: "60-key matrix / COL0..11 input with pull-ups; selected ROW low, other ROWs high-impedance"
Changed lines of the file:
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@@
 	(title_block
 		(title "WING27 / 60-key matrix")
-		(rev "electrical-2")
+		(rev "electrical-3")
 		(company "ハシビロ工業"))
 	(symbol
@@
 			(type default))
 )
+	(global_label
+"ROW_L0"
+		(shape bidirectional)
+		(at 25.4 78.74000000000001 0)
+		(effects
+			(font
+				(size 1.27 1.27))
+			(justify left))
+)
 	(wire
 		(pts
-			(xy 231.14 78.74000000000001)
+			(xy 285.75 78.74000000000001)
 			(xy 314.96 78.74000000000001))
 		(stroke
@@
 )
 	(global_label
-"ROW0"
+"ROW_R0"
 		(shape bidirectional)
-		(at 25.4 78.74000000000001 0)
+		(at 285.75 78.74000000000001 0)
 		(effects
 			(font
@@
 			(type default))
 )
+	(global_label
+"ROW_L1"
+		(shape bidirectional)
+		(at 25.4 134.62 0)
+		(effects
+			(font
+				(size 1.27 1.27))
+			(justify left))
+)
 	(wire
 		(pts
-			(xy 231.14 134.62)
+			(xy 285.75 134.62)
 			(xy 314.96 134.62))
 		(stroke
@@
 )
 	(global_label
-"ROW1"
+"ROW_R1"
 		(shape bidirectional)
-		(at 25.4 134.62 0)
+		(at 285.75 134.62 0)
 		(effects
 			(font
@@
 			(type default))
 )
+	(global_label
+"ROW_L2"
+		(shape bidirectional)
+		(at 25.4 190.5 0)
+		(effects
+			(font
+				(size 1.27 1.27))
+			(justify left))
+)
 	(wire
 		(pts
-			(xy 231.14 190.5)
+			(xy 285.75 190.5)
 			(xy 314.96 190.5))
 		(stroke
@@
 )
 	(global_label
-"ROW2"
+"ROW_R2"
 		(shape bidirectional)
-		(at 25.4 190.5 0)
+		(at 285.75 190.5 0)
 		(effects
 			(font
@@
 			(type default))
 )
+	(global_label
+"ROW_L3"
+		(shape bidirectional)
+		(at 25.4 246.38 0)
+		(effects
+			(font
+				(size 1.27 1.27))
+			(justify left))
+)
 	(wire
 		(pts
-			(xy 231.14 246.38)
+			(xy 285.75 246.38)
 			(xy 314.96 246.38))
 		(stroke
@@
 )
 	(global_label
-"ROW3"
+"ROW_R3"
 		(shape bidirectional)
-		(at 25.4 246.38 0)
+		(at 285.75 246.38 0)
 		(effects
 			(font
@@
 			(type default))
 )
+	(global_label
+"ROW_L4"
+		(shape bidirectional)
+		(at 25.4 302.26000000000005 0)
+		(effects
+			(font
+				(size 1.27 1.27))
+			(justify left))
+)
 	(wire
 		(pts
-			(xy 231.14 302.26000000000005)
+			(xy 285.75 302.26000000000005)
 			(xy 314.96 302.26000000000005))
 		(stroke
@@
 )
 	(global_label
-"ROW4"
+"ROW_R4"
 		(shape bidirectional)
-		(at 25.4 302.26000000000005 0)
+		(at 285.75 302.26000000000005 0)
 		(effects
 			(font
@@
 )
 	(text
-"60-key matrix / COL0..11 input with pull-ups; selected ROW low, other ROWs high-impedance"
+"Two independent 5x6 matrices / COL0..5 left, COL6..11 right / separate ROW_L and ROW_R"
 		(at 20.32 15.24 0)
 		(effects

Commit message: Add side LEDs and preserve verified official core routing
Other:
- added sheet Side LEDs (LEDs.kicad_sch)
Changed lines of the file:
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@@
 				(size 1.27 1.27))
 			(justify left))
-))
+)
+	(sheet
+		(at 110 350)
+		(size 90 20)
+		(fields_autoplaced yes)
+		(stroke
+			(width 0)
+			(type default))
+		(fill
+			(color 0 0 0 0))
+		(property
+"Sheetname"
+"Side LEDs"
+			(at 110 348 0)
+			(effects
+				(font
+					(size 1.27 1.27))
+				(justify left bottom)))
+		(property
+"Sheetfile"
+"LEDs.kicad_sch"
+			(at 110 372 0)
+			(effects
+				(font
+					(size 1.27 1.27))
+				(justify left top)))
+		(instances
+			(project
+"WING27"
+				(path
+"/77e26e32-63d2-500f-9544-76b2dd8b20de"
+					(page "3"))))))
